File: servo_breakout_board/shield_attempt.kicad_pcb (KiCad board)
At the start: 2 copper layers, 18 parts

Commit message: Add a copper fill to the board
Routing:
- added copper zone on B.Cu, net GND
Other:
- board outline added: 74.9 x 44.5 mm
Changed lines of the file:
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@@
-(kicad_pcb (version 4) (host pcbnew 4.0.4-stable)
+(kicad_pcb (version 4) (host pcbnew 4.0.4+e1-6308~48~ubuntu16.04.1-stable)
   (general
     (links 24)
-    (no_connects 3)
+    (no_connects 2)
     (area 149.159999 80.579999 220.933334 118.810002)
     (thickness 1.6)
-    (drawings 0)
+    (drawings 4)
     (tracks 57)
     (zones 0)
@@
   )
   (setup
-    (last_trace_width 0.5)
+    (last_trace_width 0.25)
     (user_trace_width 0.5)
     (user_trace_width 1)
@@
     )
   )
+  (gr_line (start 220.98 121.92) (end 146.05 121.92) (angle 90) (layer Edge.Cuts) (width 0.15))
+  (gr_line (start 146.05 121.92) (end 146.05 77.47) (angle 90) (layer Edge.Cuts) (width 0.15))
+  (gr_line (start 146.05 77.47) (end 220.98 77.47) (angle 90) (layer Edge.Cuts) (width 0.15))
+  (gr_line (start 220.98 77.47) (end 220.98 121.92) (angle 90) (layer Edge.Cuts) (width 0.15))
   (segment (start 179.07 90.3224) (end 179.07 111.76) (width 1) (layer F.Cu) (net 1))
   (segment (start 179.07 111.76) (end 179.07 118.11) (width 1) (layer F.Cu) (net 1))
@@
   (segment (start 158.75 93.6324) (end 158.75 87.63) (width 0.5) (layer F.Cu) (net 10))
   (segment (start 158.75 95.25) (end 158.75 93.8824) (width 0.25) (layer F.Cu) (net 10))
+  (zone (net 1) (net_name GND) (layer B.Cu) (hatch edge 0.508)
+    (connect_pads (clearance 0.508))
+    (min_thickness 0.254)
+    (fill (arc_segments 16) (thermal_gap 0.508) (thermal_bridge_width 0.508))
+    (polygon
+      (pts
+        (xy 220.98 121.92) (xy 146.05 121.92) (xy 146.05 77.47) (xy 220.98 77.47)
+      )
+    )
+  )
 )

Commit message: Second attempt at the main board
Parts:
- added ArduinoGND1: CONN_01X01, Pin_Headers:Pin_Header_Straight_1x01, F.Cu at (123.2, 95.2)
- added ArduinoVCC1: CONN_01X01, Pin_Headers:Pin_Header_Straight_1x01, F.Cu at (115.6, 95.2)
- added SENSOR1: CONN_01X01, Pin_Headers:Pin_Header_Straight_1x01, F.Cu at (111.8, 109.2)
- added SENSOR1PINS1: CONN_01X03, Pin_Headers:Pin_Header_Straight_1x03, F.Cu at (119.4, 106.7)
- added SENSOR2: CONN_01X01, Pin_Headers:Pin_Header_Straight_1x01, F.Cu at (111.8, 124.5)
- added SENSOR2PINS1: CONN_01X03, Pin_Headers:Pin_Header_Straight_1x03, F.Cu at (119.4, 121.9)
- added SENSOR3: CONN_01X01, Pin_Headers:Pin_Header_Straight_1x01, F.Cu at (91.4, 109.2)
- added SENSOR3PINS1: CONN_01X03, Pin_Headers:Pin_Header_Straight_1x03, F.Cu at (99.1, 106.7)
- added SENSOR4: CONN_01X01, Pin_Headers:Pin_Header_Straight_1x01, F.Cu at (91.4, 124.5)
- added SENSOR4PINS1: CONN_01X03, Pin_Headers:Pin_Header_Straight_1x03, F.Cu at (99.1, 121.9)
- moved LFE1 41.8 mm to (132.1, 125.7)
- moved LFEIN1 41.4 mm to (134.6, 118.1)
- moved RFEIN1 40.1 mm to (134.6, 102.9)
- moved RFE1 40.1 mm to (132.1, 95.2)
- moved LBE1 32.4 mm to (172.7, 125.7)
- moved LBEIN1 31.9 mm to (175.3, 118.1)
- moved RBE1 30.2 mm to (172.7, 95.2)
- moved RBEIN1 30.2 mm to (175.3, 102.9)
- moved ground1 19.8 mm to (201.9, 125.7)
- moved LFS1 17.3 mm to (146.1, 125.7)
- moved LFSIN1 16.3 mm to (148.6, 118.1)
- moved vcc1 15.9 mm to (201.9, 95.2)
- moved LBS1 14.0 mm to (186.7, 125.7)
- moved LBSIN1 12.7 mm to (189.2, 118.1)
- moved RFS1 12.7 mm to (146.1, 95.2)
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Routing:
- net GND: track 191.1 -> 395.6 mm
- net +5V: track 231.3 -> 415.5 mm
- net Net-(SENSOR4-Pad1): track 0.00 -> 7.62 mm
- net Net-(SENSOR3-Pad1): track 0.00 -> 7.62 mm
- net Net-(SENSOR2-Pad1): track 0.00 -> 7.62 mm
- net Net-(SENSOR1-Pad1): track 0.00 -> 7.62 mm
- net Net-(RFS1-Pad2): track 8.99 -> 7.62 mm
- net Net-(LFS1-Pad2): track 6.35 -> 7.62 mm
- net Net-(LFE1-Pad2): track 6.35 -> 7.62 mm
- net Net-(LBS1-Pad2): track 6.35 -> 7.62 mm
- net Net-(LBE1-Pad2): track 6.35 -> 7.62 mm
Other:
- board size 74.9 x 44.5 mm -> 137.2 x 68.6 mm
