File: servo_breakout_board/shield_attempt.sch (KiCad schematic (older format))
At the start: 18 parts

Commit message: Second attempt at the main board
Parts:
- added ArduinoGND1, ArduinoVCC1, SENSOR1, SENSOR2, SENSOR3, SENSOR4: CONN_01X01, Pin_Headers:Pin_Header_Straight_1x01, symbol CONN_01X01
- added SENSOR1PINS1, SENSOR2PINS1, SENSOR3PINS1, SENSOR4PINS1: CONN_01X03, Pin_Headers:Pin_Header_Straight_1x03, symbol CONN_01X03
Connections:
- net +5V: now also ArduinoVCC1.1 (P1), SENSOR1PINS1.1 (P1), SENSOR2PINS1.1 (P1), SENSOR3PINS1.1 (P1), SENSOR4PINS1.1 (P1)
- net GND: now also ArduinoGND1.1 (P1), SENSOR1PINS1.3 (P3), SENSOR2PINS1.3 (P3), SENSOR3PINS1.3 (P3), SENSOR4PINS1.3 (P3)
- new net: SENSOR1.1 (P1), SENSOR1PINS1.2 (P2)
- new net: SENSOR2.1 (P1), SENSOR2PINS1.2 (P2)
- new net: SENSOR3.1 (P1), SENSOR3PINS1.2 (P2)
- new net: SENSOR4.1 (P1), SENSOR4PINS1.2 (P2)
Changed lines of the file:
@@
 LIBS:contrib
 LIBS:valves
-LIBS:arduino_shieldsNCL
 LIBS:shield_attempt-cache
 EELAYER 25 0
@@
 $EndComp
 Wire Wire Line
-	2550 4400 7100 4400
-Wire Wire Line
-	2550 950  7050 950
+	2550 4400 9050 4400
+Wire Wire Line
+	2550 950  9050 950
 Wire Wire Line
 	7050 950  7050 2550
@@
 Wire Wire Line
 	3000 4400 3000 4750
+$Comp
+L CONN_01X01 ArduinoVCC1
+U 1 1 582AF018
+P 2100 2100
+F 0 "ArduinoVCC1" H 2100 2200 50  0000 C CNN
+F 1 "CONN_01X01" V 2200 2100 50  0000 C CNN
+F 2 "Pin_Headers:Pin_Header_Straight_1x01" H 2100 2100 50  0001 C CNN
+F 3 "" H 2100 2100 50  0000 C CNN
+	1    2100 2100
+	1    0    0    -1
+$EndComp
+$Comp
+L CONN_01X01 ArduinoGND1
+U 1 1 582AF7E9
+P 2150 3750
+F 0 "ArduinoGND1" H 2150 3850 50  0000 C CNN
+F 1 "CONN_01X01" V 2250 3750 50  0000 C CNN
+F 2 "Pin_Headers:Pin_Header_Straight_1x01" H 2150 3750 50  0001 C CNN
+F 3 "" H 2150 3750 50  0000 C CNN
+	1    2150 3750
+	1    0    0    -1
+$EndComp
+Wire Wire Line
+	2550 4150 1950 4150
+Wire Wire Line
+	1950 4150 1950 3750
+Connection ~ 2550 4150
+Wire Wire Line
+	2550 1650 1900 1650
+Wire Wire Line
+	1900 1650 1900 2100
+Connection ~ 2550 1650
+$Comp
+L CONN_01X01 SENSOR1
+U 1 1 582B001B
+P 8300 1400
+F 0 "SENSOR1" H 8300 1500 50  0000 C CNN
+F 1 "CONN_01X01" V 8400 1400 50  0000 C CNN
+F 2 "Pin_Headers:Pin_Header_Straight_1x01" H 8300 1400 50  0001 C CNN
+F 3 "" H 8300 1400 50  0000 C CNN
+	1    8300 1400
+	1    0    0    -1
+$EndComp
+$Comp
+L CONN_01X01 SENSOR2
+U 1 1 582B056D
+P 9600 1400
+F 0 "SENSOR2" H 9600 1500 50  0000 C CNN
+F 1 "CONN_01X01" V 9700 1400 50  0000 C CNN
+F 2 "Pin_Headers:Pin_Header_Straight_1x01" H 9600 1400 50  0001 C CNN
+F 3 "" H 9600 1400 50  0000 C CNN
+	1    9600 1400
+	1    0    0    -1
+$EndComp
+$Comp
+L CONN_01X01 SENSOR3
+U 1 1 582B05F6
+P 8300 3800
+F 0 "SENSOR3" H 8300 3900 50  0000 C CNN
+F 1 "CONN_01X01" V 8400 3800 50  0000 C CNN
+F 2 "Pin_Headers:Pin_Header_Straight_1x01" H 8300 3800 50  0001 C CNN
+F 3 "" H 8300 3800 50  0000 C CNN
+	1    8300 3800
+	1    0    0    -1
+$EndComp
+$Comp
+L CONN_01X01 SENSOR4
+U 1 1 582B0E05
+P 9700 3800
+F 0 "SENSOR4" H 9700 3900 50  0000 C CNN
+F 1 "CONN_01X01" V 9800 3800 50  0000 C CNN
+F 2 "Pin_Headers:Pin_Header_Straight_1x01" H 9700 3800 50  0001 C CNN
+F 3 "" H 9700 3800 50  0000 C CNN
+	1    9700 3800
+	1    0    0    -1
+$EndComp
+$Comp
+L CONN_01X03 SENSOR1PINS1
+U 1 1 582B107C
+P 7850 1400
+F 0 "SENSOR1PINS1" H 7850 1600 50  0000 C CNN
+F 1 "CONN_01X03" V 7950 1400 50  0000 C CNN
+F 2 "Pin_Headers:Pin_Header_Straight_1x03" H 7850 1400 50  0001 C CNN
+F 3 "" H 7850 1400 50  0000 C CNN
+	1    7850 1400
+	1    0    0    -1
+$EndComp
+$Comp
+L CONN_01X03 SENSOR2PINS1
+U 1 1 582B10F9
+P 9150 1400
+F 0 "SENSOR2PINS1" H 9150 1600 50  0000 C CNN
+F 1 "CONN_01X03" V 9250 1400 50  0000 C CNN
+F 2 "Pin_Headers:Pin_Header_Straight_1x03" H 9150 1400 50  0001 C CNN
+F 3 "" H 9150 1400 50  0000 C CNN
+	1    9150 1400
+	1    0    0    -1
+$EndComp
+$Comp
+L CONN_01X03 SENSOR3PINS1
+U 1 1 582B1C38
+P 7800 3800
+F 0 "SENSOR3PINS1" H 7800 4000 50  0000 C CNN
+F 1 "CONN_01X03" V 7900 3800 50  0000 C CNN
+F 2 "Pin_Headers:Pin_Header_Straight_1x03" H 7800 3800 50  0001 C CNN
+F 3 "" H 7800 3800 50  0000 C CNN
+	1    7800 3800
+	1    0    0    -1
+$EndComp
+$Comp
+L CONN_01X03 SENSOR4PINS1
+U 1 1 582B1CB3
+P 9250 3800
+F 0 "SENSOR4PINS1" H 9250 4000 50  0000 C CNN
+F 1 "CONN_01X03" V 9350 3800 50  0000 C CNN
+F 2 "Pin_Headers:Pin_Header_Straight_1x03" H 9250 3800 50  0001 C CNN
+F 3 "" H 9250 3800 50  0000 C CNN
+	1    9250 3800
+	1    0    0    -1
+$EndComp
+Wire Wire Line
+	9500 3800 9050 3800
+Wire Wire Line
+	9400 1400 8950 1400
+Wire Wire Line
+	8100 1400 7650 1400
+Wire Wire Line
+	8100 3800 7600 3800
+Wire Wire Line
+	7650 950  7650 1300
+Connection ~ 7050 950
+Wire Wire Line
+	8950 950  8950 1300
+Connection ~ 7650 950
+Wire Wire Line
+	7600 3700 7600 950
+Connection ~ 7600 950
+Wire Wire Line
+	9050 950  9050 3700
+Connection ~ 8950 950
+Wire Wire Line
+	7600 4400 7600 3900
+Connection ~ 7100 4400
+Wire Wire Line
+	7650 4400 7650 1500
+Connection ~ 7600 4400
+Wire Wire Line
+	9050 4400 9050 3900
+Connection ~ 7650 4400
+Wire Wire Line
+	8950 1500 8950 4400
+Connection ~ 8950 4400
 $EndSCHEMATC
